Commit message: Add files via upload
Latest Commit

File: src/ricky_description/urdf/ricky.xacro (robot description, xacro)
@@ -1,12 +1,12 @@
 <?xml version='1.0'?>
 <robot name="ricky" xmlns:xacro="http://www.ros.org/wiki/xacro">
-  <xacro:include filename="$(find ricky_description)/urdf/ricky.gazebo" />
-  <xacro:include filename="$(find ricky_description)/urdf/materials.xacro" />
-  <xacro:include filename="$(find ricky_description)/urdf/macros.xacro" />
+  <xacro:include filename="$(find ricky_description)/urdf/ricky.gazebo"/>
+  <xacro:include filename="$(find ricky_description)/urdf/materials.xacro"/>
+  <xacro:include filename="$(find ricky_description)/urdf/macros.xacro"/>
   <link name='chassis'>
     <pose>0 0 0.1 0 0 0</pose>
     <inertial>
-      <mass value="10.0"/>
-      <origin xyz="0.0 0 0.1" rpy=" 0 0 0"/>
+      <mass value="20.0"/>
+      <origin xyz="0.0 0 0.0" rpy=" 0 0 0"/>
       <inertia
           ixx="0.5" ixy="0" ixz="0"
@@ -17,5 +17,5 @@
     <collision name='collision'>
       <geometry>
-        <box size=".4 .2 .1"/>
+        <box size=".4 .4 .1"/>
       </geometry>
     </collision>
@@ -23,5 +23,5 @@
       <origin xyz="0 0 0" rpy=" 0 0 0"/>
       <geometry>
-        <box size=".4 .2 .1"/>
+        <box size=".4 .4 .1"/>
       </geometry>
     </visual>

Commit message: working node

File: src/ricky_description/urdf/ricky.xacro (robot description, xacro)
@@ -1,12 +1,12 @@
 <?xml version='1.0'?>
 <robot name="ricky" xmlns:xacro="http://www.ros.org/wiki/xacro">
-  <xacro:include filename="$(find ricky_description)/urdf/ricky.gazebo" />
-  <xacro:include filename="$(find ricky_description)/urdf/materials.xacro" />
-  <xacro:include filename="$(find ricky_description)/urdf/macros.xacro" />
+  <xacro:include filename="$(find ricky_description)/urdf/ricky.gazebo"/>
+  <xacro:include filename="$(find ricky_description)/urdf/materials.xacro"/>
+  <xacro:include filename="$(find ricky_description)/urdf/macros.xacro"/>
   <link name='chassis'>
     <pose>0 0 0.1 0 0 0</pose>
     <inertial>
-      <mass value="10.0"/>
-      <origin xyz="0.0 0 0.1" rpy=" 0 0 0"/>
+      <mass value="20.0"/>
+      <origin xyz="0.0 0 0.0" rpy=" 0 0 0"/>
       <inertia
           ixx="0.5" ixy="0" ixz="0"
@@ -17,5 +17,5 @@
     <collision name='collision'>
       <geometry>
-        <box size=".4 .2 .1"/>
+        <box size=".4 .4 .1"/>
       </geometry>
     </collision>
@@ -23,5 +23,5 @@
       <origin xyz="0 0 0" rpy=" 0 0 0"/>
       <geometry>
-        <box size=".4 .2 .1"/>
+        <box size=".4 .4 .1"/>
       </geometry>
     </visual>
@@ -181,4 +181,9 @@
       <alwaysOn>true</alwaysOn>
     </plugin>
+    <plugin name="gazebo_ros_control" filename="libgazebo_ros_contol.so">
+    </plugin>
   </gazebo>
+  <gazebo reference="chassis">
+      <material>Gazebo/Green</material>
+    </gazebo>
 </robot>

Commit message: ricky new branch

File: src/ricky_description/urdf/ricky.xacro (robot description, xacro)
@@ -136,5 +136,5 @@
   <joint name="hokuyo_joint" type="fixed">
     <axis xyz="0 1 0"/>
-    <origin xyz="0 0 ${0.01+0.01+0.05}" rpy="0 0 0"/>
+    <origin xyz="-0.1 0 ${0.01+0.01+0.05}" rpy="0 0 0"/>
     <parent link="chassis"/>
     <child link="hokuyo_link"/>
@@ -150,8 +150,8 @@
         <scan>
           <horizontal>
-            <samples>360</samples>
+            <samples>720</samples>
             <resolution>1</resolution>
-            <min_angle>-3.141592653589793238</min_angle>
-            <max_angle>3.141592653589793238</max_angle>
+            <min_angle>1.57079632679</min_angle>
+            <max_angle>4.71238898038</max_angle>
           </horizontal>
         </scan>

Commit message: changes to urdf/node changes

File: src/ricky_description/urdf/ricky.xacro (robot description, xacro)
@@ -17,5 +17,5 @@
     <collision name='collision'>
       <geometry>
-        <box size=".4 .4 .1"/>
+        <box size=".4 .25 .1"/>
       </geometry>
     </collision>
@@ -23,5 +23,5 @@
       <origin xyz="0 0 0" rpy=" 0 0 0"/>
       <geometry>
-        <box size=".4 .4 .1"/>
+        <box size=".4 .25 .1"/>
       </geometry>
     </visual>
@@ -50,5 +50,5 @@
   </link>
   <link name="left_wheel">
-    <!--origin xyz="0.1 0.13 0.1" rpy="0 1.5707 1.5707"/-->
+    <!-- <origin xyz="0.1 0.13 0.1" rpy="0 1.5707 1.5707"/> -->
     <collision name="collision">
       <origin xyz="0 0 0" rpy="0 1.5707 1.5707"/>
@@ -152,6 +152,6 @@
             <samples>720</samples>
             <resolution>1</resolution>
-            <min_angle>1.57079632679</min_angle>
-            <max_angle>4.71238898038</max_angle>
+            <min_angle>1.57079994678</min_angle>
+            <max_angle>4.71239984034</max_angle>
           </horizontal>
         </scan>
